File: hw/mcu/mcu.sch (KiCad schematic (older format))
At the start: 92 parts, among them J1 RJ12, P1 CONN_01X16, P2 CONN_01X16, P3 USB_B, U1 IS64WV102416, U2 stm32f429igt6, U3 ADP5070, U4 USB3300, U5 ADP7142, U6 ADP7182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

Commit message: add pdf sch
Parts:
- P3: symbol USB_B -> USB_B-RESCUE-mcu
Connections:
- no-connect marks 8 -> 68
Changed lines of the file:
@@
 EESchema Schematic File Version 2
+LIBS:mcu-rescue
 LIBS:power
 LIBS:device
@@
 LIBS:mcu
 LIBS:mcu-cache
-EELAYER 25 0
+EELAYER 26 0
 EELAYER END
 $Descr A3 16535 11693
@@
 Connection ~ 10350 2650
 $Comp
-L USB_B P3
+L USB_B-RESCUE-mcu P3
 U 1 1 57120A50
 P 10450 1750
@@
 	0    1    1    0
 $EndComp
+NoConn ~ 3350 9100
+NoConn ~ 3350 9000
+NoConn ~ 3350 8900
+NoConn ~ 3350 8800
+NoConn ~ 3350 8700
+NoConn ~ 3350 8600
+NoConn ~ 3350 7800
+NoConn ~ 3350 7700
+NoConn ~ 3350 7600
+NoConn ~ 3350 7500
+NoConn ~ 3350 7400
+NoConn ~ 3350 7300
+NoConn ~ 3350 7200
+NoConn ~ 3350 7100
+NoConn ~ 3350 7000
+NoConn ~ 3350 6900
+NoConn ~ 3350 6100
+NoConn ~ 3350 4400
+NoConn ~ 5900 1200
+NoConn ~ 5900 1300
+NoConn ~ 5900 1400
+NoConn ~ 5900 1600
+NoConn ~ 5900 1800
+NoConn ~ 5900 1900
+NoConn ~ 5900 2000
+NoConn ~ 5900 2300
+NoConn ~ 5900 2400
+NoConn ~ 5900 2500
+NoConn ~ 5900 2600
+NoConn ~ 5900 2700
+NoConn ~ 5900 3100
+NoConn ~ 5900 3200
+NoConn ~ 5900 3300
+NoConn ~ 5900 4300
+NoConn ~ 5900 4400
+NoConn ~ 5900 4700
+NoConn ~ 5900 5000
+NoConn ~ 5900 5100
+NoConn ~ 5900 5200
+NoConn ~ 5900 5300
+NoConn ~ 5900 5400
+NoConn ~ 5900 5500
+NoConn ~ 5900 5600
+NoConn ~ 5900 5700
+NoConn ~ 5900 5800
+NoConn ~ 5900 5900
+NoConn ~ 5900 6000
+NoConn ~ 5900 6100
+NoConn ~ 5900 6500
+NoConn ~ 5900 6600
+NoConn ~ 5900 6900
+NoConn ~ 5900 7100
+NoConn ~ 5900 7200
+NoConn ~ 5900 7300
+NoConn ~ 5900 8200
+NoConn ~ 5900 8400
+NoConn ~ 5900 8500
+NoConn ~ 5900 8600
+NoConn ~ 7800 5650
+NoConn ~ 7800 5550
 $EndSCHEMATC
